File: pcb/expression faders.kicad_pcb (KiCad board)
At the start: 2 copper layers, 71.5 x 149.5 mm, 8 parts, among them SW1 RotaryEncoder_Switch, SW2 RotaryEncoder_Switch, U1 XIAO-RP2040-DIP

Commit message: update readme
Connections:
- C1 pad 2: +3V3 -> +3.3V
- U1 pad 12: +3V3 -> +3.3V
Routing:
- net +3.3V: track 25.0 -> 65.3 mm, vias 0 -> 1
- net +3V3: track 7.47 -> 0.00 mm
