File: pcb/expression faders.kicad_sch (KiCad schematic)
At the start: 8 parts, among them SW1 RotaryEncoder_Switch, SW2 RotaryEncoder_Switch, U1 XIAO-RP2040-DIP

Commit message: update readme
Connections:
- net +3V3 is gone; now on net +3.3V: C1.2, U1.12 (3V3)
Changed lines of the file:
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@@
+	)
+	(junction
+		(at 116.84 83.82)
+		(diameter 0)
+		(color 0 0 0 0)
 	)
 	(junction
@@
 	(junction
 		(at 190.5 76.2)
-		(diameter 0)
-		(color 0 0 0 0)
-	)
-	(junction
-		(at 116.84 83.82)
 		(diameter 0)
 		(color 0 0 0 0)
@@
 	)
 	(symbol
-		(lib_id "power:+3V3")
+		(lib_id "power:+3.3V")
 		(at 116.84 83.82 0)
 		(unit 1)
@@
 		(dnp no)
 		(fields_autoplaced yes)
-		(property "Reference" "#PWR03"
+		(property "Reference" "#PWR01"
 			(at 116.84 87.63 0)
 			(hide yes)
@@
 			)
 		)
-		(property "Value" "+3V3"
+		(property "Value" "+3.3V"
 			(at 116.84 78.74 0)
 			(show_name no)
@@
 			)
 		)
-		(property "Description" "Power symbol creates a global label with name \"+3V3\""
+		(property "Description" "Power symbol creates a global label with name \"+3.3V\""
 			(at 116.84 83.82 0)
 			(hide yes)
@@
 			(project "expression faders"
 				(path "/ea3d44a2-fefe-4fda-b24c-6bc4055fffd6"
-					(reference "#PWR03")
+					(reference "#PWR01")
 					(unit 1)
 				)
